File: smoke85/rgb_leds.kicad_sch (KiCad schematic)
At the start: 4 parts

Commit message: start connecting rgb leds
Parts:
- removed R24: 330, Mars_Library:R_0603, symbol Device:R
- added C11, C12, C13, C14, C15, C16, C17, C18, C19, C20, C21, C22, C23, C24, C25, C26, C27, C28, C29, C30, C31: 100n, symbol Device:C_Small
- added LED10, LED11, LED12, LED13, LED14, LED15, LED16, LED17, LED18, LED19, LED20, LED21, LED4, LED5, LED6, LED7, LED8, LED9: MX_SK6812MINI-E, PCM_marbastlib-mx:LED_MX_6028R, symbol PCM_marbastlib-mx:MX_SK6812MINI-E
Connections:
- net +5V_LED: now also LED1.1 (VDD), LED2.1 (VDD), LED3.1 (VDD), C11.1, C12.1, C13.1, C14.1, C15.1, C16.1, C17.1, C18.1, C19.1, C20.1, C21.1, C22.1, C23.1, C24.1, C25.1, C26.1, C27.1, C28.1, C29.1, C30.1, C31.1, LED10.1 (VDD), LED11.1 (VDD), LED12.1 (VDD), LED13.1 (VDD), LED14.1 (VDD), LED15.1 (VDD), LED16.1 (VDD), LED17.1 (VDD), LED18.1 (VDD), LED19.1 (VDD), LED20.1 (VDD), LED21.1 (VDD), LED4.1 (VDD), LED5.1 (VDD), LED6.1 (VDD), LED7.1 (VDD), LED8.1 (VDD), LED9.1 (VDD)
- net GND: now also C11.2, C12.2, C13.2, C14.2, C15.2, C16.2, C17.2, C18.2, C19.2, C20.2, C21.2, C22.2, C23.2, C24.2, C25.2, C26.2, C27.2, C28.2, C29.2, C30.2, C31.2, LED10.4 (VSS), LED11.4 (VSS), LED12.4 (VSS), LED13.4 (VSS), LED14.4 (VSS), LED15.4 (VSS), LED16.4 (VSS), LED17.4 (VSS), LED18.4 (VSS), LED19.4 (VSS), LED20.4 (VSS), LED21.4 (VSS), LED4.4 (VSS), LED5.4 (VSS), LED6.4 (VSS), LED7.4 (VSS), LED8.4 (VSS), LED9.4 (VSS)
- net at LED3.2 (DOUT): now also LED4.3 (DIN)
- net LED_IN renamed A2
- new net: LED19.2 (DOUT), LED20.3 (DIN)
- new net: LED18.2 (DOUT), LED19.3 (DIN)
- new net: LED11.2 (DOUT), LED12.3 (DIN)
- new net: LED10.2 (DOUT), LED11.3 (DIN)
- new net: LED14.2 (DOUT), LED15.3 (DIN)
- new net: LED13.2 (DOUT), LED14.3 (DIN)
- new net: LED20.2 (DOUT), LED21.3 (DIN)
- new net: LED6.2 (DOUT), LED7.3 (DIN)
- new net: LED5.2 (DOUT), LED6.3 (DIN)
- new net: LED4.2 (DOUT), LED5.3 (DIN)
- new net: LED16.2 (DOUT), LED17.3 (DIN)
- new net: LED15.2 (DOUT), LED16.3 (DIN)
- new net: LED8.2 (DOUT), LED9.3 (DIN)
- new net: LED7.2 (DOUT), LED8.3 (DIN)
- new net: LED17.2 (DOUT), LED18.3 (DIN)
- new net: LED10.3 (DIN), LED9.2 (DOUT)
- new net: LED12.2 (DOUT), LED13.3 (DIN)
Other:
- moved on the sheet: LED1, LED2, LED3

Commit message: wire more leds
Parts:
- added C32, C33, C34, C35, C36, C37, C38, C39, C40, C41, C42, C43, C44, C45, C46, C47, C48, C49, C50, C51, C52, C53, C54, C55, C56, C57, C58, C59, C60, C61, C62, C63, C64: 100n, symbol Device:C_Small
- added LED22, LED23, LED24, LED25, LED26, LED27, LED28, LED29, LED30, LED31, LED32, LED33, LED34, LED35, LED36, LED37, LED38, LED39, LED40, LED41, LED42, LED43, LED44, LED45, LED46, LED47, LED48, LED49, LED50, LED51, LED52, LED53, LED54, LED55, LED56: MX_SK6812MINI-E, PCM_marbastlib-mx:LED_MX_6028R, symbol PCM_marbastlib-mx:MX_SK6812MINI-E
Connections:
- net +5V_LED: now also C32.1, C33.1, C34.1, C35.1, C36.1, C37.1, C38.1, C39.1, C40.1, C41.1, C42.1, C43.1, C44.1, C45.1, C46.1, C47.1, C48.1, C49.1, C50.1, C51.1, C52.1, C53.1, C54.1, C55.1, C56.1, C57.1, C58.1, C59.1, C60.1, C61.1, C62.1, C63.1, C64.1, LED22.1 (VDD), LED23.1 (VDD), LED24.1 (VDD), LED25.1 (VDD), LED26.1 (VDD), LED27.1 (VDD), LED28.1 (VDD), LED29.1 (VDD), LED30.1 (VDD), LED31.1 (VDD), LED32.1 (VDD), LED33.1 (VDD), LED34.1 (VDD), LED35.1 (VDD), LED36.1 (VDD), LED37.1 (VDD), LED38.1 (VDD), LED39.1 (VDD), LED40.1 (VDD), LED41.1 (VDD), LED42.1 (VDD), LED43.1 (VDD), LED44.1 (VDD), LED45.1 (VDD), LED46.1 (VDD), LED47.1 (VDD), LED48.1 (VDD), LED49.1 (VDD), LED50.1 (VDD), LED51.1 (VDD), LED52.1 (VDD), LED53.1 (VDD), LED54.1 (VDD), LED55.1 (VDD), LED56.1 (VDD)
- net GND: now also C32.2, C33.2, C34.2, C35.2, C36.2, C37.2, C38.2, C39.2, C40.2, C41.2, C42.2, C43.2, C44.2, C45.2, C46.2, C47.2, C48.2, C49.2, C50.2, C51.2, C52.2, C53.2, C54.2, C55.2, C56.2, C57.2, C58.2, C59.2, C60.2, C61.2, C62.2, C63.2, C64.2, LED22.4 (VSS), LED23.4 (VSS), LED24.4 (VSS), LED25.4 (VSS), LED26.4 (VSS), LED27.4 (VSS), LED28.4 (VSS), LED29.4 (VSS), LED30.4 (VSS), LED31.4 (VSS), LED32.4 (VSS), LED33.4 (VSS), LED34.4 (VSS), LED35.4 (VSS), LED36.4 (VSS), LED37.4 (VSS), LED38.4 (VSS), LED39.4 (VSS), LED40.4 (VSS), LED41.4 (VSS), LED42.4 (VSS), LED43.4 (VSS), LED44.4 (VSS), LED45.4 (VSS), LED46.4 (VSS), LED47.4 (VSS), LED48.4 (VSS), LED49.4 (VSS), LED50.4 (VSS), LED51.4 (VSS), LED52.4 (VSS), LED53.4 (VSS), LED54.4 (VSS), LED55.4 (VSS), LED56.4 (VSS)
- net at LED21.2 (DOUT): now also LED22.3 (DIN)
- new net: LED22.2 (DOUT), LED23.3 (DIN)
- new net: LED30.2 (DOUT), LED31.3 (DIN)
- new net: LED29.2 (DOUT), LED30.3 (DIN)
- new net: LED36.2 (DOUT), LED37.3 (DIN)
- new net: LED35.2 (DOUT), LED36.3 (DIN)
- new net: LED28.2 (DOUT), LED29.3 (DIN)
- new net: LED50.2 (DOUT), LED51.3 (DIN)
- new net: LED49.2 (DOUT), LED50.3 (DIN)
- new net: LED55.2 (DOUT), LED56.3 (DIN)
- new net: LED54.2 (DOUT), LED55.3 (DIN)
- new net: LED27.2 (DOUT), LED28.3 (DIN)
- new net: LED48.2 (DOUT), LED49.3 (DIN)
- new net: LED47.2 (DOUT), LED48.3 (DIN)
- new net: LED26.2 (DOUT), LED27.3 (DIN)
- new net: LED37.2 (DOUT), LED38.3 (DIN)
- new net: LED31.2 (DOUT), LED32.3 (DIN)
- new net: LED45.2 (DOUT), LED46.3 (DIN)
- new net: LED44.2 (DOUT), LED45.3 (DIN)
- new net: LED33.2 (DOUT), LED34.3 (DIN)
- new net: LED32.2 (DOUT), LED33.3 (DIN)
- new net: LED46.2 (DOUT), LED47.3 (DIN)
- new net: LED41.2 (DOUT), LED42.3 (DIN)
- new net: LED40.2 (DOUT), LED41.3 (DIN)
- new net: LED53.2 (DOUT), LED54.3 (DIN)
- new net: LED34.2 (DOUT), LED35.3 (DIN)
- new net: LED51.2 (DOUT), LED52.3 (DIN)
- new net: LED43.2 (DOUT), LED44.3 (DIN)
- new net: LED42.2 (DOUT), LED43.3 (DIN)
- new net: LED24.2 (DOUT), LED25.3 (DIN)
- new net: LED23.2 (DOUT), LED24.3 (DIN)
- new net: LED25.2 (DOUT), LED26.3 (DIN)
- new net: LED39.2 (DOUT), LED40.3 (DIN)
- new net: LED38.2 (DOUT), LED39.3 (DIN)
- new net: LED52.2 (DOUT), LED53.3 (DIN)
Other:
- moved on the sheet: C31
